Commit message: feat: Migrate firo_description

File: firo_description/robots/firo.urdf.xacro (robot description, xacro)
@@ -5,4 +5,5 @@
   <xacro:arg name="imu_frequency" default="200.0"/>
   <xacro:arg name="stereo_fps" default="30"/>
+  <xacro:arg name="gazebo" default="False"/>
   <!-- Parse arguments -->
   <xacro:property name="calibration_path" value="$(arg calibration_path)" />
@@ -20,5 +21,5 @@
   <xacro:include filename="$(find firo_description)/urdf/wheel.urdf.xacro" />
   <xacro:include filename="$(find firo_description)/urdf/oak-d-w/oak-d-w.urdf.xacro" />
- <!-- Macro to simplify joint definition -->
+  <!-- Macro to simplify joint definition -->
   <xacro:macro name="joint" params="type:='fixed' parent:='base_link' child:='' xyz:='0 0 0' rpy:='0 0 0' axis:='0 0 1' limit_effort:='0.0' limit_velocity:='0.0'">
     <joint name="${child}_joint" type="${type}">
@@ -45,50 +46,99 @@
   <xacro:joint child="back_left_wheel" xyz="${-mechanical.wheel_base/2} ${mechanical.wheel_track/2} ${mechanical.wheel_radius}" type="continuous" axis="0 1 0" limit_effort="7.5" limit_velocity="7.5"/>
   <xacro:joint parent="torso" child="front_camera" xyz="0.3001 0 0.12845"/>
-  <transmission name="front_right_wheel_transmission">
-    <type>transmission_interface/SimpleTransmission</type>
-    <actuator name="front_right_wheel_motor">
-      <mechanicalReduction>1</mechanicalReduction>
-    </actuator>
-    <joint name="front_right_wheel_joint">
-    <hardwareInterface>hardware_interface/VelocityJointInterface</hardwareInterface>
-    </joint>
-  </transmission>
-  <transmission name="front_left_wheel_transmission">
-    <type>transmission_interface/SimpleTransmission</type>
-    <actuator name="front_left_wheel_motor">
-      <mechanicalReduction>1</mechanicalReduction>
-    </actuator>
-    <joint name="front_left_wheel_joint">
-    <hardwareInterface>hardware_interface/VelocityJointInterface</hardwareInterface>
-    </joint>
-  </transmission>
-  <transmission name="back_right_wheel_transmission">
-    <type>transmission_interface/SimpleTransmission</type>
-    <actuator name="back_right_wheel_motor">
-      <mechanicalReduction>1</mechanicalReduction>
-    </actuator>
-    <joint name="back_right_wheel_joint">
-    <hardwareInterface>hardware_interface/VelocityJointInterface</hardwareInterface>
-    </joint>
-  </transmission>
-  <transmission name="back_left_wheel_transmission">
-    <type>transmission_interface/SimpleTransmission</type>
-    <actuator name="back_left_wheel_motor">
-      <mechanicalReduction>1</mechanicalReduction>
-    </actuator>
-    <joint name="back_left_wheel_joint">
-    <hardwareInterface>hardware_interface/VelocityJointInterface</hardwareInterface>
-    </joint>
-  </transmission>
+  <xacro:if value="$(arg gazebo)">
+    <ros2_control name="GazeboSimSystem" type="system">
+      <hardware>
+        <plugin>gz_ros2_control/GazeboSimSystem</plugin>
+      </hardware>
+      <joint name="front_right_wheel_joint">
+        <command_interface name="velocity">
+          <param name="min">-7.5</param>
+          <param name="max">7.5</param>
+        </command_interface>
+        <state_interface name="position">
+          <param name="initial_value">0.0</param>
+        </state_interface>
+        <state_interface name="velocity" />
+        <state_interface name="effort"/>
+      </joint>
+      <joint name="front_left_wheel_joint">
+        <command_interface name="velocity">
+          <param name="min">-7.5</param>
+          <param name="max">7.5</param>
+        </command_interface>
+        <state_interface name="position">
+          <param name="initial_value">0.0</param>
+        </state_interface>
+        <state_interface name="velocity" />
+        <state_interface name="effort"/>
+      </joint>
+      <joint name="back_right_wheel_joint">
+        <command_interface name="velocity">
+          <param name="min">-7.5</param>
+          <param name="max">7.5</param>
+        </command_interface>
+        <state_interface name="position">
+          <param name="initial_value">0.0</param>
+        </state_interface>
+        <state_interface name="velocity" />
+        <state_interface name="effort"/>
+      </joint>
+      <joint name="back_left_wheel_joint">
+        <command_interface name="velocity">
+          <param name="min">-7.5</param>
+          <param name="max">7.5</param>
+        </command_interface>
+        <state_interface name="position">
+          <param name="initial_value">0.0</param>
+        </state_interface>
+        <state_interface name="velocity" />
+        <state_interface name="effort"/>
+      </joint>
+    </ros2_control>
+  </xacro:if>
+  <xacro:unless value="$(arg gazebo)">
+    <ros2_control name="odrive_can" type="actuator">
+      <hardware>
+        <plugin>odrive_can_driver/OdriveHardwareInterface</plugin>
+        <param name="interface">can0</param>
+      </hardware>
+      <joint name="front_right_wheel_joint">
+        <param name="node_id">10</param>
+        <param name="transmission">56.25</param>
+        <command_interface name="velocity" />
+        <state_interface name="position" />
+        <state_interface name="velocity" />
+        <state_interface name="effort"/>
+      </joint>
+      <joint name="back_right_wheel_joint">
+        <param name="node_id">11</param>
+        <param name="transmission">56.25</param>
+        <command_interface name="velocity" />
+        <state_interface name="position" />
+        <state_interface name="velocity" />
+        <state_interface name="effort"/>
+      </joint>
+      <joint name="back_left_wheel_joint">
+        <param name="node_id">12</param>
+        <param name="transmission">-56.25</param>
+        <command_interface name="velocity" />
+        <state_interface name="position" />
+        <state_interface name="velocity" />
+        <state_interface name="effort"/>
+      </joint>
+      <joint name="front_left_wheel_joint">
+        <param name="node_id">13</param>
+        <param name="transmission">-56.25</param>
+        <command_interface name="velocity" />
+        <state_interface name="position" />
+        <state_interface name="velocity" />
+        <state_interface name="effort"/>
+      </joint>
+    </ros2_control>
+  </xacro:unless>
   <gazebo>
-    <plugin name="gazebo_ros_control" filename="libgazebo_ros_control.so">
-      <robotNamespace>/</robotNamespace>
-    </plugin>
-    <plugin name="p3d_plugin" filename="libgazebo_ros_p3d.so">
-      <alwaysOn>true</alwaysOn>
-      <updateRate>100.0</updateRate>
-      <bodyName>base_link</bodyName>
-      <topicName>ground_truth</topicName>
-      <frameName>map</frameName>
+    <plugin filename="libgz_ros2_control-system.so" name="gz_ros2_control::GazeboSimROS2ControlPlugin">
+      <hold_joints>true</hold_joints>
+      <parameters>$(find firo_control)/config/controllers.yaml</parameters>
     </plugin>
   </gazebo>
